File: fpga-power-and-config.sch (KiCad schematic (older format))
At the start: 18 parts

Commit message: initial footprint assignment and VERY rough placement
Parts:
- C401, C402, C403, C404, C405, C406, C407, C408, C409, C410: renamed from C?; footprint (none) -> Capacitor_SMD:C_0402_1005Metric
- D401: renamed from D?; footprint (none) -> Diode_SMD:D_SOD-523
- R401, R402, R403, R404, R405: renamed from R?; footprint (none) -> Resistor_SMD:R_0402_1005Metric
- gave numbers to parts that had none: 2
Changed lines of the file:
@@
 $EndDescr
 $Comp
-L FPGA_Lattice:ICE40HX1K-TQ144 U?
+L FPGA_Lattice:ICE40HX1K-TQ144 U301
 U 5 1 5E153448
 P 4750 5700
-F 0 "U?" H 5100 6300 50  0000 L CNN
+F 0 "U301" H 5100 6300 50  0000 L CNN
 F 1 "ICE40HX1K-TQ144" H 3950 5100 50  0000 L CNN
 F 2 "Package_QFP:TQFP-144_20x20mm_P0.5mm" H 4750 4250 50  0001 C CNN
@@
 $EndComp
 $Comp
-L Device:C C?
+L Device:C C403
 U 1 1 5E157432
 P 5450 4800
-F 0 "C?" H 5565 4846 50  0000 L CNN
+F 0 "C403" H 5565 4846 50  0000 L CNN
 F 1 "0.1u" H 5565 4755 50  0000 L CNN
-F 2 "" H 5488 4650 50  0001 C CNN
+F 2 "Capacitor_SMD:C_0402_1005Metric" H 5488 4650 50  0001 C CNN
 F 3 "~" H 5450 4800 50  0001 C CNN
 	1    5450 4800
@@
 $EndComp
 $Comp
-L Device:C C?
+L Device:C C404
 U 1 1 5E15793B
 P 5800 4800
-F 0 "C?" H 5915 4846 50  0000 L CNN
+F 0 "C404" H 5915 4846 50  0000 L CNN
 F 1 "10u" H 5915 4755 50  0000 L CNN
-F 2 "" H 5838 4650 50  0001 C CNN
+F 2 "Capacitor_SMD:C_0402_1005Metric" H 5838 4650 50  0001 C CNN
 F 3 "~" H 5800 4800 50  0001 C CNN
 	1    5800 4800
@@
 VCCPLL
 $Comp
-L Device:D D?
+L Device:D D401
 U 1 1 5E15B065
 P 4850 4700
-F 0 "D?" V 4800 4650 50  0000 R CNN
+F 0 "D401" V 4800 4650 50  0000 R CNN
 F 1 "CDBU0520" V 4700 4650 50  0000 R CNN
-F 2 "" H 4850 4700 50  0001 C CNN
+F 2 "Diode_SMD:D_SOD-523" H 4850 4700 50  0001 C CNN
 F 3 "~" H 4850 4700 50  0001 C CNN
 	1    4850 4700
@@
 	5450 5700 5350 5700
 $Comp
-L Device:R R?
+L Device:R R404
 U 1 1 5E185A56
 P 4050 5350
-F 0 "R?" H 4120 5396 50  0000 L CNN
+F 0 "R404" H 4120 5396 50  0000 L CNN
 F 1 "10k" H 4120 5305 50  0000 L CNN
-F 2 "" V 3980 5350 50  0001 C CNN
+F 2 "Resistor_SMD:R_0402_1005Metric" V 3980 5350 50  0001 C CNN
 F 3 "~" H 4050 5350 50  0001 C CNN
 	1    4050 5350
@@
 If substituting a different SPI flash, see requirements in\n"ICE40 Programming and Configuration" document, section 9.2.\nMost specs are met by pretty much all SPI NOR flash devices,\nexcept for the start-up time requirement (tVSL <= 10 us).
 $Comp
-L Memory_Flash:W25Q32JVSS U?
+L Memory_Flash:W25Q32JVSS U401
 U 1 1 5DF6C286
 P 2400 5800
-F 0 "U?" H 2050 6150 50  0000 C CNN
+F 0 "U401" H 2050 6150 50  0000 C CNN
 F 1 "W25Q80DVSNIG" H 2750 6150 50  0000 C CNN
 F 2 "Package_SO:SOIC-8_5.23x5.23mm_P1.27mm" H 2400 5800 50  0001 C CNN
@@
 MISO
 $Comp
-L Device:R R?
+L Device:R R403
 U 1 1 5DFA2A75
 P 2700 5300
-F 0 "R?" V 2650 5450 50  0000 L CNN
+F 0 "R403" V 2650 5450 50  0000 L CNN
 F 1 "10k" V 2700 5250 50  0000 L CNN
-F 2 "" V 2630 5300 50  0001 C CNN
+F 2 "Resistor_SMD:R_0402_1005Metric" V 2630 5300 50  0001 C CNN
 F 3 "~" H 2700 5300 50  0001 C CNN
 	1    2700 5300
@@
 $EndComp
 $Comp
-L Device:R R?
+L Device:R R402
 U 1 1 5DFA2C63
 P 2700 5200
-F 0 "R?" V 2650 5350 50  0000 L CNN
+F 0 "R402" V 2650 5350 50  0000 L CNN
 F 1 "10k" V 2700 5150 50  0000 L CNN
-F 2 "" V 2630 5200 50  0001 C CNN
+F 2 "Resistor_SMD:R_0402_1005Metric" V 2630 5200 50  0001 C CNN
 F 3 "~" H 2700 5200 50  0001 C CNN
 	1    2700 5200
@@
 	4450 4900 4450 5000
 $Comp
-L Device:C C?
+L Device:C C402
 U 1 1 5DFB341D
 P 3850 4700
-F 0 "C?" H 3965 4746 50  0000 L CNN
+F 0 "C402" H 3965 4746 50  0000 L CNN
 F 1 "0.1u" H 3965 4655 50  0000 L CNN
-F 2 "" H 3888 4550 50  0001 C CNN
+F 2 "Capacitor_SMD:C_0402_1005Metric" H 3888 4550 50  0001 C CNN
 F 3 "~" H 3850 4700 50  0001 C CNN
 	1    3850 4700
@@
 	3850 4950 3850 4850
 $Comp
-L power:GND #PWR?
+L power:GND #PWR0402
 U 1 1 5DFB8E53
 P 3850 4950
-F 0 "#PWR?" H 3850 4700 50  0001 C CNN
+F 0 "#PWR0402" H 3850 4700 50  0001 C CNN
 F 1 "GND" H 3855 4777 50  0000 C CNN
 F 2 "" H 3850 4950 50  0001 C CNN
@@
 $EndComp
 $Comp
-L Device:C C?
+L Device:C C401
 U 1 1 5DFB9E75
 P 1350 5800
-F 0 "C?" H 1465 5846 50  0000 L CNN
+F 0 "C401" H 1465 5846 50  0000 L CNN
 F 1 "0.1u" H 1465 5755 50  0000 L CNN
-F 2 "" H 1388 5650 50  0001 C CNN
+F 2 "Capacitor_SMD:C_0402_1005Metric" H 1388 5650 50  0001 C CNN
 F 3 "~" H 1350 5800 50  0001 C CNN
 	1    1350 5800
@@
 	2400 6500 2400 6200
 $Comp
-L power:GND #PWR?
+L power:GND #PWR0401
 U 1 1 5DFC9CFB
 P 2400 6600
-F 0 "#PWR?" H 2400 6350 50  0001 C CNN
+F 0 "#PWR0401" H 2400 6350 50  0001 C CNN
 F 1 "GND" H 2405 6427 50  0000 C CNN
 F 2 "" H 2400 6600 50  0001 C CNN
@@
 Connection ~ 2400 6500
 $Comp
-L Device:R R?
+L Device:R R401
 U 1 1 5DFD7EEB
 P 1700 5450
-F 0 "R?" H 1770 5496 50  0000 L CNN
+F 0 "R401" H 1770 5496 50  0000 L CNN
 F 1 "10k" H 1770 5405 50  0000 L CNN
-F 2 "" V 1630 5450 50  0001 C CNN
+F 2 "Resistor_SMD:R_0402_1005Metric" V 1630 5450 50  0001 C CNN
 F 3 "~" H 1700 5450 50  0001 C CNN
 	1    1700 5450
@@
 	4750 4050 5800 4050
 $Comp
-L Device:R R?
+L Device:R R405
 U 1 1 5E07EE3A
 P 5800 4300
-F 0 "R?" H 5870 4346 50  0000 L CNN
+F 0 "R405" H 5870 4346 50  0000 L CNN
 F 1 "10k" H 5870 4255 50  0000 L CNN
-F 2 "" V 5730 4300 50  0001 C CNN
+F 2 "Resistor_SMD:R_0402_1005Metric" V 5730 4300 50  0001 C CNN
 F 3 "~" H 5800 4300 50  0001 C CNN
 	1    5800 4300
@@
 	5800 4450 5800 4550
 $Comp
-L Device:C C?
+L Device:C C405
 U 1 1 5E0953B8
 P 6250 4300
-F 0 "C?" H 6365 4346 50  0000 L CNN
+F 0 "C405" H 6365 4346 50  0000 L CNN
 F 1 "0.01u" H 6365 4255 50  0000 L CNN
-F 2 "" H 6288 4150 50  0001 C CNN
+F 2 "Capacitor_SMD:C_0402_1005Metric" H 6288 4150 50  0001 C CNN
 F 3 "~" H 6250 4300 50  0001 C CNN
 	1    6250 4300
@@
 $EndComp
 $Comp
-L Device:C C?
+L Device:C C406
 U 1 1 5E0958B9
 P 6650 4300
-F 0 "C?" H 6765 4346 50  0000 L CNN
+F 0 "C406" H 6765 4346 50  0000 L CNN
 F 1 "0.1u" H 6765 4255 50  0000 L CNN
-F 2 "" H 6688 4150 50  0001 C CNN
+F 2 "Capacitor_SMD:C_0402_1005Metric" H 6688 4150 50  0001 C CNN
 F 3 "~" H 6650 4300 50  0001 C CNN
 	1    6650 4300
@@
 $EndComp
 $Comp
-L Device:C C?
+L Device:C C407
 U 1 1 5E095E61
 P 7050 4300
-F 0 "C?" H 7165 4346 50  0000 L CNN
+F 0 "C407" H 7165 4346 50  0000 L CNN
 F 1 "0.1u" H 7165 4255 50  0000 L CNN
-F 2 "" H 7088 4150 50  0001 C CNN
+F 2 "Capacitor_SMD:C_0402_1005Metric" H 7088 4150 50  0001 C CNN
 F 3 "~" H 7050 4300 50  0001 C CNN
 	1    7050 4300
@@
 $EndComp
 $Comp
-L Device:C C?
+L Device:C C408
 U 1 1 5E096291
 P 7450 4300
-F 0 "C?" H 7565 4346 50  0000 L CNN
+F 0 "C408" H 7565 4346 50  0000 L CNN
 F 1 "0.1u" H 7565 4255 50  0000 L CNN
-F 2 "" H 7488 4150 50  0001 C CNN
+F 2 "Capacitor_SMD:C_0402_1005Metric" H 7488 4150 50  0001 C CNN
 F 3 "~" H 7450 4300 50  0001 C CNN
 	1    7450 4300
@@
 $EndComp
 $Comp
-L Device:C C?
+L Device:C C409
 U 1 1 5E09DD35
 P 7850 4300
-F 0 "C?" H 7965 4346 50  0000 L CNN
+F 0 "C409" H 7965 4346 50  0000 L CNN
 F 1 "0.1u" H 7965 4255 50  0000 L CNN
-F 2 "" H 7888 4150 50  0001 C CNN
+F 2 "Capacitor_SMD:C_0402_1005Metric" H 7888 4150 50  0001 C CNN
 F 3 "~" H 7850 4300 50  0001 C CNN
 	1    7850 4300
@@
 $EndComp
 $Comp
-L Device:C C?
+L Device:C C410
 U 1 1 5E09DECE
 P 8250 4300
-F 0 "C?" H 8365 4346 50  0000 L CNN
+F 0 "C410" H 8365 4346 50  0000 L CNN
 F 1 "10u" H 8365 4255 50  0000 L CNN
-F 2 "" H 8288 4150 50  0001 C CNN
+F 2 "Capacitor_SMD:C_0402_1005Metric" H 8288 4150 50  0001 C CNN
 F 3 "~" H 8250 4300 50  0001 C CNN
 	1    8250 4300
@@
 	7850 4550 7450 4550
 $Comp
-L power:GND #PWR?
+L power:GND #PWR0404
 U 1 1 5E0CCB0A
 P 8250 4650
-F 0 "#PWR?" H 8250 4400 50  0001 C CNN
+F 0 "#PWR0404" H 8250 4400 50  0001 C CNN
 F 1 "GND" H 8255 4477 50  0000 C CNN
 F 2 "" H 8250 4650 50  0001 C CNN
@@
 Connection ~ 8250 4550
 $Comp
-L power:GND #PWR?
+L power:GND #PWR0403
 U 1 1 5E0D30AD
 P 4750 6500
-F 0 "#PWR?" H 4750 6250 50  0001 C CNN
+F 0 "#PWR0403" H 4750 6250 50  0001 C CNN
 F 1 "GND" H 4755 6327 50  0000 C CNN
 F 2 "" H 4750 6500 50  0001 C CNN

Commit message: local component placement
Parts:
- R405: value 10k -> 100
Changed lines of the file:
@@
 P 5800 4300
 F 0 "R405" H 5870 4346 50  0000 L CNN
-F 1 "10k" H 5870 4255 50  0000 L CNN
+F 1 "100" H 5870 4255 50  0000 L CNN
 F 2 "Resistor_SMD:R_0402_1005Metric" V 5730 4300 50  0001 C CNN
 F 3 "~" H 5800 4300 50  0001 C CNN
