File: m2-conn.sch (KiCad schematic (older format))
At the start: 1 part

Commit message: initial footprint assignment and VERY rough placement
Parts:
- added J602: M.2-GND-MOUNTING, symbol Connector_Generic:Conn_01x01
- J601: renamed from J??; footprint (none) -> m2ngff:m2-padKeyB
Connections:
- net GND: now also J602.1 (Pin_1)
Changed lines of the file:
@@
 $EndDescr
 $Comp
-L m2:m.2_socket2_module J??
+L m2:m.2_socket2_module J601
 U 1 1 5DF7ABC6
 P 2900 1750
-F 0 "J??" H 3625 1915 50  0000 C CNN
+F 0 "J601" H 3625 1915 50  0000 C CNN
 F 1 "m.2_socket2_module" H 3625 1824 50  0000 C CNN
-F 2 "" H 2850 2000 50  0001 C CNN
+F 2 "m2ngff:m2-padKeyB" H 2850 2000 50  0001 C CNN
 F 3 "" H 2850 2000 50  0001 C CNN
 	1    2900 1750
@@
 	4700 5050 4450 5050
 $Comp
-L power:GND #PWR?
+L power:GND #PWR0601
 U 1 1 5DF7C006
 P 4550 5450
-F 0 "#PWR?" H 4550 5200 50  0001 C CNN
+F 0 "#PWR0601" H 4550 5200 50  0001 C CNN
 F 1 "GND" H 4555 5277 50  0000 C CNN
 F 2 "" H 4550 5450 50  0001 C CNN
@@
 Text HLabel 2600 1900 0    50   Output ~ 0
 3.3V
+$Comp
+L Connector_Generic:Conn_01x01 J602
+U 1 1 5DF8F75E
+P 6750 2000
+F 0 "J602" H 6830 2042 50  0000 L CNN
+F 1 "M.2-GND-MOUNTING" H 6830 1951 50  0000 L CNN
+F 2 "" H 6750 2000 50  0001 C CNN
+F 3 "~" H 6750 2000 50  0001 C CNN
+	1    6750 2000
+	1    0    0    -1
+$EndComp
+$Comp
+L power:GND #PWR0602
+U 1 1 5DF8FED9
+P 6450 2100
+F 0 "#PWR0602" H 6450 1850 50  0001 C CNN
+F 1 "GND" H 6455 1927 50  0000 C CNN
+F 2 "" H 6450 2100 50  0001 C CNN
+F 3 "" H 6450 2100 50  0001 C CNN
+	1    6450 2100
+	1    0    0    -1
+$EndComp
+Wire Wire Line
+	6450 2100 6450 2000
+Wire Wire Line
+	6450 2000 6550 2000
 $EndSCHEMATC

Commit message: added a couple more footprints
Parts:
- J602: footprint (none) -> m2-ice40:m.2_mechanical_ground_pad
Changed lines of the file:
@@
 F 0 "J602" H 6830 2042 50  0000 L CNN
 F 1 "M.2-GND-MOUNTING" H 6830 1951 50  0000 L CNN
-F 2 "" H 6750 2000 50  0001 C CNN
+F 2 "m2-ice40:m.2_mechanical_ground_pad" H 6750 2000 50  0001 C CNN
 F 3 "~" H 6750 2000 50  0001 C CNN
 	1    6750 2000
