File: power.sch (KiCad schematic (older format))
At the start: 11 parts

Commit message: initial footprint assignment and VERY rough placement
Parts:
- C501, C502, C503, C504: renamed from C?; footprint (none) -> Capacitor_SMD:C_0402_1005Metric
- R501, R502, R503, R504, R505: renamed from R?; footprint (none) -> Resistor_SMD:R_0402_1005Metric
- TP501: renamed from TP?; footprint (none) -> TestPoint:TestPoint_Pad_1.0x1.0mm
- gave numbers to parts that had none: 1
Changed lines of the file:
@@
 $Descr A4 11693 8268
 encoding utf-8
-Sheet 6 7
+Sheet 5 7
 Title ""
 Date ""
@@
 $EndDescr
 $Comp
-L m2:TPSM82822 U?
+L m2:TPSM82822 U501
 U 1 1 5E141E34
 P 5000 2000
-F 0 "U?" H 5350 2165 50  0000 C CNN
+F 0 "U501" H 5350 2165 50  0000 C CNN
 F 1 "TPSM82821" H 5350 2074 50  0000 C CNN
 F 2 "" H 5000 2000 50  0001 C CNN
@@
 $EndComp
 $Comp
-L Device:C C?
+L Device:C C501
 U 1 1 5E141E3A
 P 4500 2500
-F 0 "C?" H 4615 2546 50  0000 L CNN
+F 0 "C501" H 4615 2546 50  0000 L CNN
 F 1 "4.7u" H 4615 2455 50  0000 L CNN
-F 2 "" H 4538 2350 50  0001 C CNN
+F 2 "Capacitor_SMD:C_0402_1005Metric" H 4538 2350 50  0001 C CNN
 F 3 "~" H 4500 2500 50  0001 C CNN
 	1    4500 2500
@@
 $EndComp
 $Comp
-L Device:C C?
+L Device:C C504
 U 1 1 5E141E40
 P 7650 2600
-F 0 "C?" H 7765 2646 50  0000 L CNN
+F 0 "C504" H 7765 2646 50  0000 L CNN
 F 1 "10u" H 7765 2555 50  0000 L CNN
-F 2 "" H 7688 2450 50  0001 C CNN
+F 2 "Capacitor_SMD:C_0402_1005Metric" H 7688 2450 50  0001 C CNN
 F 3 "~" H 7650 2600 50  0001 C CNN
 	1    7650 2600
@@
 $EndComp
 $Comp
-L Device:C C?
+L Device:C C503
 U 1 1 5E141E46
 P 7250 2600
-F 0 "C?" H 7365 2646 50  0000 L CNN
+F 0 "C503" H 7365 2646 50  0000 L CNN
 F 1 "10u" H 7365 2555 50  0000 L CNN
-F 2 "" H 7288 2450 50  0001 C CNN
+F 2 "Capacitor_SMD:C_0402_1005Metric" H 7288 2450 50  0001 C CNN
 F 3 "~" H 7250 2600 50  0001 C CNN
 	1    7250 2600
@@
 $EndComp
 $Comp
-L Device:R R?
+L Device:R R504
 U 1 1 5E141E4C
 P 6500 2350
-F 0 "R?" H 6570 2396 50  0000 L CNN
+F 0 "R504" H 6570 2396 50  0000 L CNN
 F 1 "100k" H 6570 2305 50  0000 L CNN
-F 2 "" V 6430 2350 50  0001 C CNN
+F 2 "Resistor_SMD:R_0402_1005Metric" V 6430 2350 50  0001 C CNN
 F 3 "~" H 6500 2350 50  0001 C CNN
 	1    6500 2350
@@
 $EndComp
 $Comp
-L Device:R R?
+L Device:R R505
 U 1 1 5E141E52
 P 6500 2850
-F 0 "R?" H 6570 2896 50  0000 L CNN
+F 0 "R505" H 6570 2896 50  0000 L CNN
 F 1 "100k" H 6570 2805 50  0000 L CNN
-F 2 "" V 6430 2850 50  0001 C CNN
+F 2 "Resistor_SMD:R_0402_1005Metric" V 6430 2850 50  0001 C CNN
 F 3 "~" H 6500 2850 50  0001 C CNN
 	1    6500 2850
@@
 $EndComp
 $Comp
-L Device:C C?
+L Device:C C502
 U 1 1 5E141E58
 P 6850 2350
-F 0 "C?" H 6965 2396 50  0000 L CNN
+F 0 "C502" H 6965 2396 50  0000 L CNN
 F 1 "120p" H 6965 2305 50  0000 L CNN
-F 2 "" H 6888 2200 50  0001 C CNN
+F 2 "Capacitor_SMD:C_0402_1005Metric" H 6888 2200 50  0001 C CNN
 F 3 "~" H 6850 2350 50  0001 C CNN
 	1    6850 2350
@@
 Connection ~ 7650 2100
 $Comp
-L Device:R R?
+L Device:R R503
 U 1 1 5E141E79
 P 6150 2850
-F 0 "R?" H 6220 2896 50  0000 L CNN
+F 0 "R503" H 6220 2896 50  0000 L CNN
 F 1 "100k" H 6220 2805 50  0000 L CNN
-F 2 "" V 6080 2850 50  0001 C CNN
+F 2 "Resistor_SMD:R_0402_1005Metric" V 6080 2850 50  0001 C CNN
 F 3 "~" H 6150 2850 50  0001 C CNN
 	1    6150 2850
@@
 3.3V_M.2
 $Comp
-L Device:R R?
+L Device:R R501
 U 1 1 5E144877
 P 3250 1500
-F 0 "R?" V 3150 1500 50  0000 C CNN
+F 0 "R501" V 3150 1500 50  0000 C CNN
 F 1 "0" V 3250 1500 50  0000 C CNN
-F 2 "" V 3180 1500 50  0001 C CNN
+F 2 "Resistor_SMD:R_0402_1005Metric" V 3180 1500 50  0001 C CNN
 F 3 "~" H 3250 1500 50  0001 C CNN
 	1    3250 1500
@@
 $EndComp
 $Comp
-L Device:R R?
+L Device:R R502
 U 1 1 5E144C04
 P 3250 1700
-F 0 "R?" V 3150 1700 50  0000 C CNN
+F 0 "R502" V 3150 1700 50  0000 C CNN
 F 1 "0" V 3250 1700 50  0000 C CNN
-F 2 "" V 3180 1700 50  0001 C CNN
+F 2 "Resistor_SMD:R_0402_1005Metric" V 3180 1700 50  0001 C CNN
 F 3 "~" H 3250 1700 50  0001 C CNN
 F 4 "DNP" V 3350 1700 50  0000 C CNN "Note"
@@
 	3100 1700 3000 1700
 $Comp
-L Connector:TestPoint TP?
+L Connector:TestPoint TP501
 U 1 1 5E149EF0
 P 3000 1700
-F 0 "TP?" V 3000 2000 50  0000 C CNN
+F 0 "TP501" V 3000 2000 50  0000 C CNN
 F 1 "3.3V_EXT" V 2900 1900 50  0000 C CNN
-F 2 "" H 3200 1700 50  0001 C CNN
+F 2 "TestPoint:TestPoint_Pad_1.0x1.0mm" H 3200 1700 50  0001 C CNN
 F 3 "~" H 3200 1700 50  0001 C CNN
 	1    3000 1700

Commit message: added a couple more footprints
Parts:
- U501: footprint (none) -> m2-ice40:SIL0010D
Changed lines of the file:
@@
 F 0 "U501" H 5350 2165 50  0000 C CNN
 F 1 "TPSM82821" H 5350 2074 50  0000 C CNN
-F 2 "" H 5000 2000 50  0001 C CNN
+F 2 "m2-ice40:SIL0010D" H 5000 2000 50  0001 C CNN
 F 3 "" H 5000 2000 50  0001 C CNN
 	1    5000 2000

Commit message: local component placement
Connections:
- net GND: now reaches C501.2, C503.2, C504.2, R505.2, U501.10 (GND), U501.9 (GND)
Changed lines of the file:
@@
 Text Label 4200 2100 0    50   ~ 0
 3.3V
+$Comp
+L power:GND #PWR0101
+U 1 1 5E0D6090
+P 4800 3300
+F 0 "#PWR0101" H 4800 3050 50  0001 C CNN
+F 1 "GND" H 4805 3127 50  0000 C CNN
+F 2 "" H 4800 3300 50  0001 C CNN
+F 3 "" H 4800 3300 50  0001 C CNN
+	1    4800 3300
+	1    0    0    -1
+$EndComp
+Wire Wire Line
+	4800 3300 4800 3200
 $EndSCHEMATC
